Commit message: fix: extend thumb proximal joint limits for retargeting
The th_proximal_link joint at q=0 already has ~34° bend due to the
joint origin. With lower limit at 0, the optimizer could never
straighten the thumb, causing it to always saturate at max bend.

Extend lower limit to -0.5 (distal mimic to -0.35) so the optimizer
can produce both straight and bent thumb poses.

File: robots/hands/rohand/rohand_right.urdf (robot description, URDF)
Before this commit: robot rohand_right, 18 links, 17 joints
Joints:
- joint th_distal_link: limit lower=0 upper=0.7 effort=0 velocity=0 -> lower=-0.35 upper=0.7 effort=0 velocity=0
- joint th_proximal_link: limit lower=0 upper=1.0 effort=0 velocity=0 -> lower=-0.5 upper=1.0 effort=0 velocity=0

Commit message: fix: correct finger joint limits to [-1.57, 0] for proper retargeting
Finger joints close in the negative direction. The symmetric [-1.57, 1.57]
limits allowed the optimizer into the positive (hyperextension) range,
causing half-bent poses when the hand should be fully open (q=0).

Also keeps th_proximal extended range [-0.5, 1.0] for thumb bending.

File: robots/hands/rohand/rohand_right.urdf (robot description, URDF)
Before this commit: robot rohand_right, 18 links, 17 joints
Joints:
- joint if_distal_link: limit lower=-1.57 upper=1.57 effort=0 velocity=0 -> lower=-1.57 upper=0 effort=0 velocity=0
- joint if_proximal_link: limit lower=-1.57 upper=1.57 effort=0 velocity=0 -> lower=-1.57 upper=0 effort=0 velocity=0
- joint lf_distal_link: limit lower=-1.57 upper=1.57 effort=0 velocity=0 -> lower=-1.57 upper=0 effort=0 velocity=0
- joint lf_proximal_link: limit lower=-1.57 upper=1.57 effort=0 velocity=0 -> lower=-1.57 upper=0 effort=0 velocity=0
- joint mf_distal_link: limit lower=-1.57 upper=1.57 effort=0 velocity=0 -> lower=-1.57 upper=0 effort=0 velocity=0
- joint mf_proximal_link: limit lower=-1.57 upper=1.57 effort=0 velocity=0 -> lower=-1.57 upper=0 effort=0 velocity=0
- joint rf_distal_link: limit lower=-1.57 upper=1.57 effort=0 velocity=0 -> lower=-1.57 upper=0 effort=0 velocity=0
- joint rf_proximal_link: limit lower=-1.57 upper=1.57 effort=0 velocity=0 -> lower=-1.57 upper=0 effort=0 velocity=0
